File: ulx4m-cm4-hat.kicad_pcb (KiCad board)
At the start: 2 copper layers, 65 x 56 mm, 5 parts, among them J1 Raspberry_Pi_2_3

Commit message: Version v1.0
Parts:
- added C1: 100n, Capacitor_SMD:C_0603_1608Metric, F.Cu at (123.4, 86.8)
- added C10: 100n, Capacitor_SMD:C_0603_1608Metric, F.Cu at (144.0, 85.7)
- added C11: 10n, Capacitor_SMD:C_0603_1608Metric, F.Cu at (144.0, 87.3)
- added C2: 10n, Capacitor_SMD:C_0603_1608Metric, F.Cu at (125.0, 86.8)
- added C21: 22uF, Capacitor_SMD:C_0805_2012Metric, F.Cu at (121.5, 87.0)
- added C3: 22uF, Capacitor_SMD:C_0805_2012Metric, F.Cu at (153.8, 61.8)
- added C4: 100n, Capacitor_SMD:C_0603_1608Metric, F.Cu at (154.0, 63.6)
- added C5: 10n, Capacitor_SMD:C_0603_1608Metric, F.Cu at (154.0, 65.3)
- added C6: 100n, Capacitor_SMD:C_0603_1608Metric, F.Cu at (154.0, 67.5)
- added C7: 10n, Capacitor_SMD:C_0603_1608Metric, F.Cu at (154.0, 69.1)
- added C8: 22uF, Capacitor_SMD:C_0805_2012Metric, F.Cu at (153.8, 71.0)
- added C9: 22uF, Capacitor_SMD:C_0805_2012Metric, F.Cu at (144.2, 83.8)
- added D1: R, LED_SMD:LED_0805_2012Metric, F.Cu at (136.1, 95.6)
- added D2: B, LED_SMD:LED_0805_2012Metric, F.Cu at (139.1, 95.6)
- added D3: G, LED_SMD:LED_0805_2012Metric, F.Cu at (142.1, 95.6)
- added D4: R, LED_SMD:LED_0805_2012Metric, F.Cu at (145.1, 95.6)
- added J4: CONN_02X03, Connector_PinSocket_2.54mm:PinSocket_2x03_P2.54mm_Vertical, F.Cu at (153.5, 82.6)
- added R1: 549, Resistor_SMD:R_0603_1608Metric, F.Cu at (136.3, 92.2)
- added R2: 549, Resistor_SMD:R_0603_1608Metric, F.Cu at (139.3, 92.2)
- added R3: 1K, Resistor_SMD:R_0603_1608Metric, F.Cu at (145.3, 102.2)
- added R34: 15k, Resistor_SMD:R_0603_1608Metric, F.Cu at (127.3, 102.2)
- added R35: 549, Resistor_SMD:R_0603_1608Metric, F.Cu at (135.3, 102.2)
- added R4: 1K, Resistor_SMD:R_0603_1608Metric, F.Cu at (155.3, 102.2)
- added R49: 27, Resistor_SMD:R_0603_1608Metric, F.Cu at (122.8, 91.7)
- added R5: 549, Resistor_SMD:R_0603_1608Metric, F.Cu at (142.3, 92.2)
- added R50: 27, Resistor_SMD:R_0603_1608Metric, F.Cu at (122.8, 93.2)
- added R56: 15k, Resistor_SMD:R_0603_1608Metric, F.Cu at (146.6, 72.1)
- added R6: 549, Resistor_SMD:R_0603_1608Metric, F.Cu at (145.3, 92.2)
- added R9: 15k, Resistor_SMD:R_0603_1608Metric, F.Cu at (146.6, 73.8)
- added SW1: WIFI ENABLE, Switch_EVPAA:Switch_EVPAA, F.Cu at (131.3, 101.8)
- added SW2: BTN2, Switch_EVPAA:Switch_EVPAA, F.Cu at (141.3, 101.9)
- added SW3: BTN1, Switch_EVPAA:Switch_EVPAA, F.Cu at (151.3, 101.9)
- added U1: LM1117-3.3, Package_TO_SOT_SMD:SOT-223-3_TabPin2, F.Cu at (145.1, 67.5)
- added U2: FT231XS, ft231x:FT231X-SSOP-20_4.4x6.5mm_Pitch0.65mm, F.Cu at (144.8, 79.0)
- added U9: ESP32, ESP32:ESP32, F.Cu at (121.9, 72.2)
- added US1: MICRO_USB, usb_otg:USB-MICRO-B-FCI-10118192-0001LF, F.Cu at (114.8, 91.7)
Connections:
- J1 pad 1: (no net) -> +3V3
- J1 pad 10: (no net) -> SD_CLK
- J1 pad 11: (no net) -> WIFI_GPIO35
- J1 pad 12: (no net) -> RP_GPIO18
- J1 pad 13: (no net) -> SD_CMD
- J1 pad 14: (no net) -> GND
- J1 pad 15: (no net) -> WIFI_EN
- J1 pad 16: (no net) -> FTDI_TXD
- J1 pad 17: (no net) -> +3V3
- J1 pad 18: (no net) -> FTDI_RXD
- J1 pad 19: (no net) -> WIFI_GPIO26
- J1 pad 2: (no net) -> +5V
- J1 pad 20: (no net) -> GND
- J1 pad 21: (no net) -> WIFI_GPIO27
- J1 pad 22: (no net) -> WIFI_TXD
- J1 pad 23: (no net) -> WIFI_GPIO25
- J1 pad 24: (no net) -> WIFI_GPIO19
- J1 pad 25: (no net) -> GND
- J1 pad 26: (no net) -> RP_GPIO07
- J1 pad 27: (no net) -> WIFI_GPIO21
- J1 pad 28: (no net) -> WIFI_GPIO22
- J1 pad 29: (no net) -> WIFI_GPIO33
- J1 pad 3: (no net) -> SD_D2
- J1 pad 30: (no net) -> GND
- J1 pad 31: (no net) -> RP_GPIO06
- J1 pad 32: (no net) -> JTAG_TDI
- J1 pad 33: (no net) -> FTDI_TXDEN
- J1 pad 34: (no net) -> GND
- J1 pad 35: (no net) -> WIFI_GPIO0
- J1 pad 36: (no net) -> JTAG_TDO
- J1 pad 37: (no net) -> WIFI_RXD
- J1 pad 38: (no net) -> JTAG_TCK
- J1 pad 39: (no net) -> GND
- J1 pad 4: (no net) -> +5V
- J1 pad 40: (no net) -> JTAG_TMS
- J1 pad 5: (no net) -> SD_D1
- J1 pad 6: (no net) -> GND
- J1 pad 7: (no net) -> SD_D0
- J1 pad 8: (no net) -> SD_D3
- J1 pad 9: (no net) -> GND
Routing:
- net +3V3: track 0.00 -> 213.7 mm, vias 0 -> 5
- net GND: track 0.00 -> 172.6 mm, vias 0 -> 47
- net +5V: track 0.00 -> 126.7 mm, vias 0 -> 1
- net JTAG_TMS: track 0.00 -> 110.4 mm, vias 0 -> 2
- net JTAG_TDI: track 0.00 -> 86.3 mm, vias 0 -> 2
- net JTAG_TCK: track 0.00 -> 86.1 mm, vias 0 -> 3
- net JTAG_TDO: track 0.00 -> 85.4 mm, vias 0 -> 3
- net USB_FTDI_D+: track 0.00 -> 78.1 mm
- net USB_FTDI_D-: track 0.00 -> 77.8 mm
- net RP_GPIO07: track 0.00 -> 69.5 mm, vias 0 -> 2
- net WIFI_GPIO0: track 0.00 -> 67.0 mm, vias 0 -> 3
- net WIFI_GPIO33: track 0.00 -> 58.4 mm, vias 0 -> 2
- net RP_GPIO06: track 0.00 -> 58.2 mm, vias 0 -> 2
- net WIFI_EN: track 0.00 -> 57.2 mm
- net WIFI_RXD: track 0.00 -> 51.9 mm, vias 0 -> 1
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- added copper zone on F.Cu, net GND
- added copper zone on In1.Cu, net GND
- added copper zone on In2.Cu, net GND
Other:
- copper layers 2 -> 4
- board text removed: "Mounting holes H5 and H6 line up with mounting holes on the Pi 3"
