File: ulx4m-cm4-hat.sch (KiCad schematic (older format))
At the start: 7 parts, among them J1 Raspberry_Pi_2_3, J3 WIFI_OFF, U9 ESP32

Commit message: Version v1.0
Parts:
- removed J3: WIFI_OFF, Connector_PinHeader_2.54mm:PinHeader_1x02_P2.54mm_Vertical, symbol Connector_Generic:Conn_02x01
- added C1, C10, C4, C6: 100n, Capacitor_SMD:C_0603_1608Metric, symbol Device:C
- added C11, C2, C5, C7: 10n, Capacitor_SMD:C_0603_1608Metric, symbol Device:C
- added C3, C8, C9: 22uF, Capacitor_SMD:C_0805_2012Metric, symbol Device:C
- added D1, D4: R, LED_SMD:LED_0805_2012Metric, symbol Device:LED_Small
- added D2: B, LED_SMD:LED_0805_2012Metric, symbol Device:LED_Small
- added D3: G, LED_SMD:LED_0805_2012Metric, symbol Device:LED_Small
- added J4: CONN_02X03, Connector_PinSocket_2.54mm:PinSocket_2x03_P2.54mm_Vertical, symbol Connector_Generic:Conn_02x03_Odd_Even
- added R1, R2, R5, R6: 549, Resistor_SMD:R_0603_1608Metric, symbol Device:R
- added R3, R4: 1K, Resistor_SMD:R_0603_1608Metric, symbol Device:R
- added R49, R50: 27, Resistor_SMD:R_0603_1608Metric, symbol Device:R
- added R9: 15k, Resistor_SMD:R_0603_1608Metric, symbol Device:R
- added SW1: WIFI ENABLE, Switch_EVPAA:Switch_EVPAA, symbol Switch:SW_Push
- added SW2: BTN2, Switch_EVPAA:Switch_EVPAA, symbol Switch:SW_Push
- added SW3: BTN1, Switch_EVPAA:Switch_EVPAA, symbol Switch:SW_Push
- added U1: LM1117-3.3, Package_TO_SOT_SMD:SOT-223-3_TabPin2, symbol Regulator_Linear:LM1117-3.3
- added U2: FT231XS, ft231x:FT231X-SSOP-20_4.4x6.5mm_Pitch0.65mm, symbol ftdi:FT231XS
- added US1: MICRO_USB, usb_otg:USB-MICRO-B-FCI-10118192-0001LF, symbol usb_otg:USB_OTG
Connections:
- net GP12 is gone; now on net WIFI_GPIO33: U9.9 (IO33)
- net +3V3: now also C1.1, C10.1, C11.1, C2.1, C6.1, C7.1, C8.1, C9.1, D2.2 (A), D3.2 (A), D4.2 (A), J4.2 (Pin_2), R3.1, R4.1, R9.2, U1.2 (VO), U2.3 (VCCIO)
- net GND: now also J1.14 (GND), J1.20 (GND), J1.25 (GND), J1.30 (GND), J1.34 (GND), J1.39 (GND), J1.6 (GND), J1.9 (GND), C1.2, C10.2, C11.2, C2.2, C3.2, C4.2, C5.2, C6.2, C7.2, C8.2, C9.2, J4.1 (Pin_1), R1.2, SW1.2, U1.1 (GND), U2.16 (GND), U2.6 (GND), US1.5 (GND), US1.6 (shield)
- net JTAG_TCK: now also J4.4 (Pin_4), U2.7 (~DSR)
- net JTAG_TDI: now also J4.3 (Pin_3), U2.5 (~RI)
- net JTAG_TDO: now also J4.6 (Pin_6), U2.9 (~CTS)
- net JTAG_TMS: now also J4.5 (Pin_5), R6.1, U2.8 (~DCD)
- net WIFIEN: now also SW1.1
- net WIFI_EN: now also J1.15 (GPIO22)
- net WIFI_GPIO0: now also J1.35 (GPIO19/MISO1)
- net WIFI_GPIO19: now also J1.24 (~CE0~/GPIO8)
- net WIFI_GPIO21: now also J1.27 (ID_SD/GPIO0)
- net WIFI_GPIO22: now also J1.28 (ID_SC/GPIO1)
- net WIFI_GPIO25: now also J1.23 (SCLK0/GPIO11)
- net WIFI_GPIO26: now also J1.19 (MOSI0/GPIO10)
- net WIFI_GPIO27: now also J1.21 (MISO0/GPIO9)
- net WIFI_GPIO35: now also J1.11 (GPIO17)
- net WIFI_RXD: now also J1.37 (GPIO26)
- net WIFI_TXD: now also J1.22 (GPIO25)
- net RP_GPIO18: now reaches J1.12 (GPIO18/PWM0)
- net RP_GPIO18: now also D1.2 (A)
- net FTDI_TXD: now reaches J1.16 (GPIO23)
- net FTDI_TXD: now also U2.20 (TXD)
- net FTDI_RXD: now reaches J1.18 (GPIO24)
- net FTDI_RXD: now also U2.4 (RXD)
- net +5V: now reaches J1.2 (5V)
- net +5V: now also J1.4 (5V), C3.1, C4.1, C5.1, U1.3 (VI), U2.15 (VCC), US1.1 (VBUS)
- net RP_GPIO07: now reaches J1.26 (~CE1~/GPIO7)
- net RP_GPIO07: now also SW2.2
- net WIFI_GPIO33: now reaches J1.29 (GCLK1/GPIO5)
- net RP_GPIO06: now reaches J1.31 (GCLK2/GPIO6)
- net RP_GPIO06: now also SW3.2
- net FTDI_TXDEN: now reaches J1.33 (PWM1/GPIO13)
- net FTDI_TXDEN: now also U2.18 (CBUS0)
- net GN12 renamed WIFI_GPIO32
- net GN13 renamed WIFI_SENSOR_VN
- net GP13 renamed WIFI_SENSOR_VP
- new net: D1.1 (K), R1.1
- new net: R4.2, SW3.1
- new net: R3.2, SW2.1
- new net: D2.1 (K), R2.2
- new net: D3.1 (K), R5.2
- new net: D4.1 (K), R6.2
- new net FTD+: R50.2, US1.3 (D+)
- new net FTD-: R49.2, US1.2 (D-)
- new net FTDI_nDTR: U2.1 (~DTR)
- new net FTDI_nRTS: U2.2 (~RTS)
- new net FTDI_nRXLED: R2.1, U2.17 (CBUS1)
- new net FTDI_nSLEEP: U2.19 (CBUS3)
- new net FTDI_nTXLED: R5.1, U2.10 (CBUS2)
- new net USB_FTDI_D+: R50.1, U2.11 (USBDP)
- new net USB_FTDI_D-: R49.1, U2.12 (USBDM)
- new net nRESET: R9.1, U2.14 (~RESET)
- no-connect marks 2 -> 3
Other:
- note added: "D8,D9: Schottky 2A/30V \nLow drop Vfmax=0.375V\nParts reduction: Only D8 is required.\nD9 D51 D52 can be 1206\n1A polyfuses or 0-ohm/2A jumpers"
- note added: "STPS2L40AF"
- moved on the sheet: C21, J1, R34, R35, R56, U9
